File: house.kicad_sch (KiCad schematic)
At the start: 10 parts, among them U5 LMR36510ADDA

Commit message: Renumber refdes
Parts:
- renumbered C55 to C31, C56 to C32, C57 to C33, C58 to C34, C59 to C35, C60 to C36, C61 to C37, L5 to L2, R31 to R16, U5 to U3
Changed lines of the file:
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@@
 		(dnp no)
 		(fields_autoplaced yes)
-		(property "Reference" "C57"
+		(property "Reference" "C33"
 			(at 119.38 92.7162 0)
 			(effects
@@
 			(project "huskypointofload"
 				(path "/eb9c972b-d134-41da-be97-ece3f463f7e0/ba0a2c31-2b64-4688-8bc7-8fc63c7eca77"
-					(reference "C64")
-					(unit 1)
-				)
-				(path "/eb9c972b-d134-41da-be97-ece3f463f7e0/c7be17f0-832c-4fd9-a896-8c518f3eba26"
-					(reference "C57")
+					(reference "C40")
+					(unit 1)
+				)
+				(path "/eb9c972b-d134-41da-be97-ece3f463f7e0/c7be17f0-832c-4fd9-a896-8c518f3eba26"
+					(reference "C33")
 					(unit 1)
 				)
@@
 		(on_board yes)
 		(dnp no)
-		(property "Reference" "C55"
+		(property "Reference" "C31"
 			(at 100.33 82.5562 0)
 			(effects
@@
 			(project "huskypointofload"
 				(path "/eb9c972b-d134-41da-be97-ece3f463f7e0/ba0a2c31-2b64-4688-8bc7-8fc63c7eca77"
-					(reference "C62")
-					(unit 1)
-				)
-				(path "/eb9c972b-d134-41da-be97-ece3f463f7e0/c7be17f0-832c-4fd9-a896-8c518f3eba26"
-					(reference "C55")
+					(reference "C38")
+					(unit 1)
+				)
+				(path "/eb9c972b-d134-41da-be97-ece3f463f7e0/c7be17f0-832c-4fd9-a896-8c518f3eba26"
+					(reference "C31")
 					(unit 1)
 				)
@@
 		(dnp no)
 		(fields_autoplaced yes)
-		(property "Reference" "C60"
+		(property "Reference" "C36"
 			(at 172.72 85.0962 0)
 			(effects
@@
 			(project "huskypointofload"
 				(path "/eb9c972b-d134-41da-be97-ece3f463f7e0/ba0a2c31-2b64-4688-8bc7-8fc63c7eca77"
-					(reference "C67")
-					(unit 1)
-				)
-				(path "/eb9c972b-d134-41da-be97-ece3f463f7e0/c7be17f0-832c-4fd9-a896-8c518f3eba26"
-					(reference "C60")
+					(reference "C43")
+					(unit 1)
+				)
+				(path "/eb9c972b-d134-41da-be97-ece3f463f7e0/c7be17f0-832c-4fd9-a896-8c518f3eba26"
+					(reference "C36")
 					(unit 1)
 				)
@@
 		(dnp no)
 		(fields_autoplaced yes)
-		(property "Reference" "C61"
+		(property "Reference" "C37"
 			(at 181.61 85.0962 0)
 			(effects
@@
 			(project "huskypointofload"
 				(path "/eb9c972b-d134-41da-be97-ece3f463f7e0/ba0a2c31-2b64-4688-8bc7-8fc63c7eca77"
-					(reference "C68")
-					(unit 1)
-				)
-				(path "/eb9c972b-d134-41da-be97-ece3f463f7e0/c7be17f0-832c-4fd9-a896-8c518f3eba26"
-					(reference "C61")
+					(reference "C44")
+					(unit 1)
+				)
+				(path "/eb9c972b-d134-41da-be97-ece3f463f7e0/c7be17f0-832c-4fd9-a896-8c518f3eba26"
+					(reference "C37")
 					(unit 1)
 				)
@@
 		(dnp no)
 		(fields_autoplaced yes)
-		(property "Reference" "U5"
+		(property "Reference" "U3"
 			(at 130.81 71.12 0)
 			(effects
@@
 			(project "huskypointofload"
 				(path "/eb9c972b-d134-41da-be97-ece3f463f7e0/ba0a2c31-2b64-4688-8bc7-8fc63c7eca77"
-					(reference "U6")
-					(unit 1)
-				)
-				(path "/eb9c972b-d134-41da-be97-ece3f463f7e0/c7be17f0-832c-4fd9-a896-8c518f3eba26"
-					(reference "U5")
+					(reference "U4")
+					(unit 1)
+				)
+				(path "/eb9c972b-d134-41da-be97-ece3f463f7e0/c7be17f0-832c-4fd9-a896-8c518f3eba26"
+					(reference "U3")
 					(unit 1)
 				)
@@
 		(dnp no)
 		(fields_autoplaced yes)
-		(property "Reference" "R31"
+		(property "Reference" "R16"
 			(at 151.13 90.1699 0)
 			(effects
@@
 			(project "huskypointofload"
 				(path "/eb9c972b-d134-41da-be97-ece3f463f7e0/ba0a2c31-2b64-4688-8bc7-8fc63c7eca77"
-					(reference "R32")
-					(unit 1)
-				)
-				(path "/eb9c972b-d134-41da-be97-ece3f463f7e0/c7be17f0-832c-4fd9-a896-8c518f3eba26"
-					(reference "R31")
+					(reference "R17")
+					(unit 1)
+				)
+				(path "/eb9c972b-d134-41da-be97-ece3f463f7e0/c7be17f0-832c-4fd9-a896-8c518f3eba26"
+					(reference "R16")
 					(unit 1)
 				)
@@
 		(dnp no)
 		(fields_autoplaced yes)
-		(property "Reference" "C58"
+		(property "Reference" "C34"
 			(at 146.0563 72.39 90)
 			(effects
@@
 			(project "huskypointofload"
 				(path "/eb9c972b-d134-41da-be97-ece3f463f7e0/ba0a2c31-2b64-4688-8bc7-8fc63c7eca77"
-					(reference "C65")
-					(unit 1)
-				)
-				(path "/eb9c972b-d134-41da-be97-ece3f463f7e0/c7be17f0-832c-4fd9-a896-8c518f3eba26"
-					(reference "C58")
+					(reference "C41")
+					(unit 1)
+				)
+				(path "/eb9c972b-d134-41da-be97-ece3f463f7e0/c7be17f0-832c-4fd9-a896-8c518f3eba26"
+					(reference "C34")
 					(unit 1)
 				)
@@
 		(dnp no)
 		(fields_autoplaced yes)
-		(property "Reference" "C59"
+		(property "Reference" "C35"
 			(at 163.83 85.0962 0)
 			(effects
@@
 			(project "huskypointofload"
 				(path "/eb9c972b-d134-41da-be97-ece3f463f7e0/ba0a2c31-2b64-4688-8bc7-8fc63c7eca77"
-					(reference "C66")
-					(unit 1)
-				)
-				(path "/eb9c972b-d134-41da-be97-ece3f463f7e0/c7be17f0-832c-4fd9-a896-8c518f3eba26"
-					(reference "C59")
+					(reference "C42")
+					(unit 1)
+				)
+				(path "/eb9c972b-d134-41da-be97-ece3f463f7e0/c7be17f0-832c-4fd9-a896-8c518f3eba26"
+					(reference "C35")
 					(unit 1)
 				)
@@
 		(dnp no)
 		(fields_autoplaced yes)
-		(property "Reference" "#PWR074"
+		(property "Reference" "#PWR037"
 			(at 130.81 107.95 0)
 			(effects
@@
 			(project "huskypointofload"
 				(path "/eb9c972b-d134-41da-be97-ece3f463f7e0/ba0a2c31-2b64-4688-8bc7-8fc63c7eca77"
-					(reference "#PWR075")
-					(unit 1)
-				)
-				(path "/eb9c972b-d134-41da-be97-ece3f463f7e0/c7be17f0-832c-4fd9-a896-8c518f3eba26"
-					(reference "#PWR074")
+					(reference "#PWR038")
+					(unit 1)
+				)
+				(path "/eb9c972b-d134-41da-be97-ece3f463f7e0/c7be17f0-832c-4fd9-a896-8c518f3eba26"
+					(reference "#PWR037")
 					(unit 1)
 				)
@@
 		(dnp no)
 		(fields_autoplaced yes)
-		(property "Reference" "L5"
+		(property "Reference" "L2"
 			(at 156.21 76.2 90)
 			(effects
@@
 			(project "huskypointofload"
 				(path "/eb9c972b-d134-41da-be97-ece3f463f7e0/ba0a2c31-2b64-4688-8bc7-8fc63c7eca77"
-					(reference "L6")
-					(unit 1)
-				)
-				(path "/eb9c972b-d134-41da-be97-ece3f463f7e0/c7be17f0-832c-4fd9-a896-8c518f3eba26"
-					(reference "L5")
+					(reference "L3")
+					(unit 1)
+				)
+				(path "/eb9c972b-d134-41da-be97-ece3f463f7e0/c7be17f0-832c-4fd9-a896-8c518f3eba26"
+					(reference "L2")
 					(unit 1)
 				)
@@
 		(dnp no)
 		(fields_autoplaced yes)
-		(property "Reference" "C56"
+		(property "Reference" "C32"
 			(at 110.49 82.5562 0)
 			(effects
@@
 			(project "huskypointofload"
 				(path "/eb9c972b-d134-41da-be97-ece3f463f7e0/ba0a2c31-2b64-4688-8bc7-8fc63c7eca77"
-					(reference "C63")
-					(unit 1)
-				)
-				(path "/eb9c972b-d134-41da-be97-ece3f463f7e0/c7be17f0-832c-4fd9-a896-8c518f3eba26"
-					(reference "C56")
-					(unit 1)
-				)
+					(reference "C39")
+					(unit 1)
+				)
+				(path "/eb9c972b-d134-41da-be97-ece3f463f7e0/c7be17f0-832c-4fd9-a896-8c518f3eba26"
+					(reference "C32")
+					(unit 1)
+				)
