File: buffer_10MHz.kicad_sch (KiCad schematic)
At the start: 23 parts

Commit message: Renumber refdes
Parts:
- renumbered C96 to C86, C97 to C87, C95 to C88, C94 to C89, C88 to C91, C87 to C92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

Commit message: Add LMX Draft
Parts:
- renumbered R38 to R40, R39 to R41, R40 to R42, R41 to R43, R42 to R44, R43 to R45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
