File: dist10.kicad_sch (KiCad schematic)
At the start: 11 parts, among them U13 LM7171xIM

Commit message: Renumber refdes
Parts:
- renumbered C89 to C81, C98 to C82, C101 to C83, C99 to C84, C100 to C85, R52 to R33, R55 to R34, R56 to R35, R57 to R36, R58 to R37, U13 to U10
Changed lines of the file:
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@@
 		(dnp no)
 		(fields_autoplaced yes)
-		(property "Reference" "#PWR0108"
+		(property "Reference" "#PWR078"
 			(at 86.36 83.82 0)
 			(effects
@@
 			(project "huskypointofload"
 				(path "/eb9c972b-d134-41da-be97-ece3f463f7e0/afb00c68-0259-43f8-a90b-9aecb9e48121"
-					(reference "#PWR0108")
+					(reference "#PWR078")
 					(unit 1)
 				)
@@
 		(dnp no)
 		(fields_autoplaced yes)
-		(property "Reference" "C99"
+		(property "Reference" "C84"
 			(at 107.95 113.0362 0)
 			(effects
@@
 			(project "huskypointofload"
 				(path "/eb9c972b-d134-41da-be97-ece3f463f7e0/afb00c68-0259-43f8-a90b-9aecb9e48121"
-					(reference "C99")
+					(reference "C84")
 					(unit 1)
 				)
@@
 		(on_board yes)
 		(dnp no)
-		(property "Reference" "#PWR0109"
+		(property "Reference" "#PWR079"
 			(at 86.36 121.92 0)
 			(effects
@@
 			(project "huskypointofload"
 				(path "/eb9c972b-d134-41da-be97-ece3f463f7e0/afb00c68-0259-43f8-a90b-9aecb9e48121"
-					(reference "#PWR0109")
+					(reference "#PWR079")
 					(unit 1)
 				)
@@
 		(on_board yes)
 		(dnp no)
-		(property "Reference" "C101"
+		(property "Reference" "C83"
 			(at 99.06 146.0562 0)
 			(effects
@@
 			(project "huskypointofload"
 				(path "/eb9c972b-d134-41da-be97-ece3f463f7e0/afb00c68-0259-43f8-a90b-9aecb9e48121"
-					(reference "C101")
+					(reference "C83")
 					(unit 1)
 				)
@@
 		(on_board yes)
 		(dnp yes)
-		(property "Reference" "R55"
+		(property "Reference" "R34"
 			(at 67.31 135.8899 0)
 			(effects
@@
 			(project "huskypointofload"
 				(path "/eb9c972b-d134-41da-be97-ece3f463f7e0/afb00c68-0259-43f8-a90b-9aecb9e48121"
-					(reference "R55")
+					(reference "R34")
 					(unit 1)
 				)
@@
 		(dnp no)
 		(fields_autoplaced yes)
-		(property "Reference" "C100"
+		(property "Reference" "C85"
 			(at 107.95 133.3562 0)
 			(effects
@@
 			(project "huskypointofload"
 				(path "/eb9c972b-d134-41da-be97-ece3f463f7e0/afb00c68-0259-43f8-a90b-9aecb9e48121"
-					(reference "C100")
+					(reference "C85")
 					(unit 1)
 				)
@@
 		(on_board yes)
 		(dnp no)
-		(property "Reference" "C98"
+		(property "Reference" "C82"
 			(at 80.0163 86.36 90)
 			(effects
@@
 			(project "huskypointofload"
 				(path "/eb9c972b-d134-41da-be97-ece3f463f7e0/afb00c68-0259-43f8-a90b-9aecb9e48121"
-					(reference "C98")
+					(reference "C82")
 					(unit 1)
 				)
@@
 		(dnp no)
 		(fields_autoplaced yes)
-		(property "Reference" "R52"
+		(property "Reference" "R33"
 			(at 62.23 96.52 90)
 			(effects
@@
 			(project "huskypointofload"
 				(path "/eb9c972b-d134-41da-be97-ece3f463f7e0/afb00c68-0259-43f8-a90b-9aecb9e48121"
-					(reference "R52")
+					(reference "R33")
 					(unit 1)
 				)
@@
 		(on_board yes)
 		(dnp no)
-		(property "Reference" "#PWR0107"
+		(property "Reference" "#PWR077"
 			(at 69.85 161.29 0)
 			(effects
@@
 			(project "huskypointofload"
 				(path "/eb9c972b-d134-41da-be97-ece3f463f7e0/afb00c68-0259-43f8-a90b-9aecb9e48121"
-					(reference "#PWR0107")
+					(reference "#PWR077")
 					(unit 1)
 				)
@@
 		(on_board yes)
 		(dnp no)
-		(property "Reference" "#PWR0106"
+		(property "Reference" "#PWR076"
 			(at 69.85 101.6 0)
 			(effects
@@
 			(project "huskypointofload"
 				(path "/eb9c972b-d134-41da-be97-ece3f463f7e0/afb00c68-0259-43f8-a90b-9aecb9e48121"
-					(reference "#PWR0106")
+					(reference "#PWR076")
 					(unit 1)
 				)
@@
 		(dnp no)
 		(fields_autoplaced yes)
-		(property "Reference" "R56"
+		(property "Reference" "R35"
 			(at 88.9 85.0899 0)
 			(effects
@@
 			(project "huskypointofload"
 				(path "/eb9c972b-d134-41da-be97-ece3f463f7e0/afb00c68-0259-43f8-a90b-9aecb9e48121"
-					(reference "R56")
+					(reference "R35")
 					(unit 1)
 				)
@@
 		(on_board yes)
 		(dnp no)
-		(property "Reference" "#PWR0110"
+		(property "Reference" "#PWR080"
 			(at 101.6 161.29 0)
 			(effects
@@
 			(project "huskypointofload"
 				(path "/eb9c972b-d134-41da-be97-ece3f463f7e0/afb00c68-0259-43f8-a90b-9aecb9e48121"
-					(reference "#PWR0110")
+					(reference "#PWR080")
 					(unit 1)
 				)
@@
 		(on_board yes)
 		(dnp no)
-		(property "Reference" "R58"
+		(property "Reference" "R37"
 			(at 99.06 133.3499 0)
 			(effects
@@
 			(project "huskypointofload"
 				(path "/eb9c972b-d134-41da-be97-ece3f463f7e0/afb00c68-0259-43f8-a90b-9aecb9e48121"
-					(reference "R58")
+					(reference "R37")
 					(unit 1)
 				)
@@
 		(on_board yes)
 		(dnp yes)
-		(property "Reference" "C89"
+		(property "Reference" "C81"
 			(at 67.31 146.0562 0)
 			(effects
@@
 			(project "huskypointofload"
 				(path "/eb9c972b-d134-41da-be97-ece3f463f7e0/afb00c68-0259-43f8-a90b-9aecb9e48121"
-					(reference "C89")
+					(reference "C81")
 					(unit 1)
 				)
@@
 		(on_board yes)
 		(dnp no)
-		(property "Reference" "R57"
+		(property "Reference" "R36"
 			(at 99.06 113.0299 0)
 			(effects
@@
 			(project "huskypointofload"
 				(path "/eb9c972b-d134-41da-be97-ece3f463f7e0/afb00c68-0259-43f8-a90b-9aecb9e48121"
-					(reference "R57")
+					(reference "R36")
 					(unit 1)
 				)
@@
 		(dnp no)
 		(fields_autoplaced yes)
-		(property "Reference" "U13"
+		(property "Reference" "U10"
 			(at 100.33 97.7198 0)
 			(effects
@@
 			(project "huskypointofload"
 				(path "/eb9c972b-d134-41da-be97-ece3f463f7e0/afb00c68-0259-43f8-a90b-9aecb9e48121"
-					(reference "U13")
-					(unit 1)
-				)
+					(reference "U10")
+					(unit 1)
+				)

Commit message: Add LMX Draft
Parts:
- renumbered R33 to R35, R34 to R36, R35 to R37, R36 to R38, R37 to R39
Changed lines of the file:
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@@
 		(dnp no)
 		(fields_autoplaced yes)
-		(property "Reference" "#PWR078"
+		(property "Reference" "#PWR079"
 			(at 86.36 83.82 0)
 			(effects
@@
 			(project "huskypointofload"
 				(path "/eb9c972b-d134-41da-be97-ece3f463f7e0/afb00c68-0259-43f8-a90b-9aecb9e48121"
-					(reference "#PWR078")
+					(reference "#PWR079")
 					(unit 1)
 				)
@@
 		(on_board yes)
 		(dnp no)
-		(property "Reference" "#PWR079"
+		(property "Reference" "#PWR080"
 			(at 86.36 121.92 0)
 			(effects
@@
 			(project "huskypointofload"
 				(path "/eb9c972b-d134-41da-be97-ece3f463f7e0/afb00c68-0259-43f8-a90b-9aecb9e48121"
-					(reference "#PWR079")
+					(reference "#PWR080")
 					(unit 1)
 				)
@@
 		(on_board yes)
 		(dnp yes)
-		(property "Reference" "R34"
+		(property "Reference" "R36"
 			(at 67.31 135.8899 0)
 			(effects
@@
 			(project "huskypointofload"
 				(path "/eb9c972b-d134-41da-be97-ece3f463f7e0/afb00c68-0259-43f8-a90b-9aecb9e48121"
-					(reference "R34")
+					(reference "R36")
 					(unit 1)
 				)
@@
 		(dnp no)
 		(fields_autoplaced yes)
-		(property "Reference" "R33"
+		(property "Reference" "R35"
 			(at 62.23 96.52 90)
 			(effects
@@
 			(project "huskypointofload"
 				(path "/eb9c972b-d134-41da-be97-ece3f463f7e0/afb00c68-0259-43f8-a90b-9aecb9e48121"
-					(reference "R33")
+					(reference "R35")
 					(unit 1)
 				)
@@
 		(on_board yes)
 		(dnp no)
-		(property "Reference" "#PWR077"
+		(property "Reference" "#PWR078"
 			(at 69.85 161.29 0)
 			(effects
@@
 			(project "huskypointofload"
 				(path "/eb9c972b-d134-41da-be97-ece3f463f7e0/afb00c68-0259-43f8-a90b-9aecb9e48121"
-					(reference "#PWR077")
+					(reference "#PWR078")
 					(unit 1)
 				)
@@
 		(on_board yes)
 		(dnp no)
-		(property "Reference" "#PWR076"
+		(property "Reference" "#PWR077"
 			(at 69.85 101.6 0)
 			(effects
@@
 			(project "huskypointofload"
 				(path "/eb9c972b-d134-41da-be97-ece3f463f7e0/afb00c68-0259-43f8-a90b-9aecb9e48121"
-					(reference "#PWR076")
+					(reference "#PWR077")
 					(unit 1)
 				)
@@
 		(dnp no)
 		(fields_autoplaced yes)
-		(property "Reference" "R35"
+		(property "Reference" "R37"
 			(at 88.9 85.0899 0)
 			(effects
@@
 			(project "huskypointofload"
 				(path "/eb9c972b-d134-41da-be97-ece3f463f7e0/afb00c68-0259-43f8-a90b-9aecb9e48121"
-					(reference "R35")
+					(reference "R37")
 					(unit 1)
 				)
@@
 		(on_board yes)
 		(dnp no)
-		(property "Reference" "#PWR080"
+		(property "Reference" "#PWR081"
 			(at 101.6 161.29 0)
 			(effects
@@
 			(project "huskypointofload"
 				(path "/eb9c972b-d134-41da-be97-ece3f463f7e0/afb00c68-0259-43f8-a90b-9aecb9e48121"
-					(reference "#PWR080")
+					(reference "#PWR081")
 					(unit 1)
 				)
@@
 		(on_board yes)
 		(dnp no)
-		(property "Reference" "R37"
+		(property "Reference" "R39"
 			(at 99.06 133.3499 0)
 			(effects
@@
 			(project "huskypointofload"
 				(path "/eb9c972b-d134-41da-be97-ece3f463f7e0/afb00c68-0259-43f8-a90b-9aecb9e48121"
-					(reference "R37")
+					(reference "R39")
 					(unit 1)
 				)
@@
 		(on_board yes)
 		(dnp no)
-		(property "Reference" "R36"
+		(property "Reference" "R38"
 			(at 99.06 113.0299 0)
 			(effects
@@
 			(project "huskypointofload"
 				(path "/eb9c972b-d134-41da-be97-ece3f463f7e0/afb00c68-0259-43f8-a90b-9aecb9e48121"
-					(reference "R36")
-					(unit 1)
-				)
+					(reference "R38")
+					(unit 1)
+				)
