File: hf_output.kicad_sch (KiCad schematic)
At the start: 9 parts, among them J16 SMP_P, J17 SMP_N

Commit message: Add LMX Draft
Parts:
- renumbered R133 to R139, R134 to R140, R135 to R141, R136 to R142, R137 to R143
