File: hf_output.kicad_sch (KiCad schematic)
At the start: 9 parts, among them J16 SMP_P, J17 SMP_N

Commit message: For Darrel
Parts:
- renumbered C173 to C112, C174 to C113, J16 to J23, J17 to J24, R139 to R130, R140 to R131, R141 to R132, R142 to R133, R143 to R134

Commit message: Add Clock sources and monitor output
Parts:
- J27: renamed from J23; value SMP_P -> MMCX_P
- J28: renamed from J24; value SMP_N -> MMCX_N
- renumbered C112 to C116, C113 to C117, R130 to R115, R131 to R116, R132 to R117, R133 to R118, R134 to R119

Commit message: Round 1 review comments
Parts:
- renumbered C116 to C150, C117 to C151, J27 to J30, J28 to J31, R115 to R168, R116 to R169, R117 to R170, R118 to R171, R119 to R172

Commit message: Round 2 Review, power tree cleanup
Parts:
- renumbered C150 to C152, C151 to C153, J30 to J31, J31 to J32, R168 to R180, R169 to R181, R170 to R182, R171 to R183, R172 to R184

Commit message: Passive footprint pass
Parts:
- R180, R181, R182, R183, R184: footprint (none) -> Resistor_SMD:R_0402_1005Metric
Changed lines of the file:
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@@
 			)
 		)
-		(property "Footprint" ""
+		(property "Footprint" "Resistor_SMD:R_0402_1005Metric"
 			(at 137.16 92.71 0)
 			(hide yes)
@@
 			)
 		)
-		(property "Footprint" ""
+		(property "Footprint" "Resistor_SMD:R_0402_1005Metric"
 			(at 86.36 92.71 0)
 			(hide yes)
@@
 			)
 		)
-		(property "Footprint" ""
+		(property "Footprint" "Resistor_SMD:R_0402_1005Metric"
 			(at 106.68 81.28 0)
 			(hide yes)
@@
 			)
 		)
-		(property "Footprint" ""
+		(property "Footprint" "Resistor_SMD:R_0402_1005Metric"
 			(at 91.44 92.71 0)
 			(hide yes)
@@
 			)
 		)
-		(property "Footprint" ""
+		(property "Footprint" "Resistor_SMD:R_0402_1005Metric"
 			(at 142.24 92.71 0)
 			(hide yes)
