File: lf_balun_output.kicad_sch (KiCad schematic)
At the start: 15 parts, among them J28 Conn_Coaxial_Small

Commit message: Add LMX Draft
Parts:
- renumbered R163 to R169, R164 to R170, R165 to R171, R166 to R172, R167 to R173, R168 to R174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
