File: lmk04828.kicad_sch (KiCad schematic)
At the start: 64 parts, among them U18 XX-XXX-VVXXFFF.fffff, U19 LMK0482x, Y2 ASE-xxxMHz

Commit message: Complete LMK schematic
Parts:
- added C160: 22p, symbol Device:C_Small
- added C161: 2.2n, symbol Device:C_Small
- added C164: 10u, symbol Device:C_Small
- added C165: 100n, symbol Device:C_Small
- added C166, C167, C168, C169: 100n, Capacitor_SMD:C_0402_1005Metric, symbol Device:C_Small
- added R116: 2.7k, symbol Device:R_Small
- added R126, R127, R128, R129: 240, symbol Device:R_Small
- renumbered C144 to C137, C137 to C138, C138 to C139, C139 to C140, C140 to C141, C141 to C142, C142 to C143, C143 to C144, C148 to C146, C146 to C147, C147 to C148, C160 to C162, C161 to C163, R116 to R117, R117 to R118, R118 to R119, R119 to R120, R120 to R121, R121 to R122, R122 to R123, R123 to R124, R124 to R125
Connections:
- net GND: now also C160.2, C164.2, C165.2, R116.2, R126.2, R127.2, R128.2, R129.2
- net at U19.1 (DCLK0_{P}): now also C166.1
- net at U19.11 (LDOBYP_{1}): now also C164.1
- net at U19.12 (LDOBYP_{2}): now also C165.1
- net HF Out 3/C+: now reaches U19.13 (SDCLK3_{P})
- net HF Out 3/C-: now reaches U19.14 (SDCLK3_{N})
- net HF Out 2/C+: now reaches U19.15 (DCLK2_{P})
- net HF Out 2/C-: now reaches U19.16 (DCLK2_{N})
- net at U19.2 (DCLK0_{N}): now also C167.1
- net HF Out 5/C+: now reaches U19.22 (SDCLK5_{P})
- net HF Out 5/C-: now reaches U19.23 (SDCLK5_{N})
- net HF Out 4/C+: now reaches U19.24 (DCLK4_{P})
- net HF Out 4/C-: now reaches U19.25 (DCLK4_{N})
- net HF Out 6/C+: now reaches U19.27 (DCLK6_{P})
- net HF Out 6/C-: now reaches U19.28 (DCLK6_{N})
- net HF Out 7/C+: now reaches U19.29 (SDCLK7_{P})
- net at U19.3 (SDCLK1_{P}): now also C168.1
- net HF Out 7/C-: now reaches U19.30 (SDCLK7_{N})
- net at U19.32 (CP_{1}): now also C160.1, C161.1
- net at U19.4 (SDCLK1_{N}): now also C169.1
- net LF Balun Output 9/C+: now reaches U19.49 (SDCLK9_{P})
- net LF Balun Output 9/C-: now reaches U19.50 (SDCLK9_{N})
- net LF Balun Output 8/C+: now reaches U19.51 (DCLK8_{P})
- net LF Balun Output 8/C-: now reaches U19.52 (DCLK8_{N})
- net LF Balun Output 10/C+: now reaches U19.54 (DCLK10_{P})
- net LF Balun Output 10/C-: now reaches U19.55 (DCLK10_{N})
- net LF Balun Output 11/C+: now reaches U19.56 (SDCLK11_{P})
- net LF Balun Output 11/C-: now reaches U19.57 (SDCLK11_{N})
- new net: C161.2, R116.1
- new net DCLK0n: C167.2, R126.1
- new net DCLK0p: C166.2, R128.1
- new net SDCLK1n: C169.2, R127.1
- new net SDCLK1p: C168.2, R129.1
Other:
- added sheet HF Out 2 (hf_output.kicad_sch)
- added sheet HF Out 3 (hf_output.kicad_sch)
- added sheet HF Out 4 (hf_output.kicad_sch)
- added sheet HF Out 5 (hf_output.kicad_sch)
- added sheet HF Out 6 (hf_output.kicad_sch)
- added sheet HF Out 7 (hf_output.kicad_sch)
- added sheet LF Balun Output 10 (lf_balun_output.kicad_sch)
- added sheet LF Balun Output 11 (lf_balun_output.kicad_sch)
- added sheet LF Balun Output 8 (lf_balun_output.kicad_sch)
- added sheet LF Balun Output 9 (lf_balun_output.kicad_sch)
- moved on the sheet: C137, C145, C146, C156, C157, C158, C159, C162, C163, R100, R101, R102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

Commit message: Add LMX Draft
Parts:
- C167: now fitted
- C169: now not fitted
- R132: renamed from R126; now fitted
- R133: renamed from R127; now not fitted
- R134: renamed from R128; now fitted
- R135: renamed from R129; now not fitted
- renumbered R94 to R100, R95 to R101, R96 to R102, R97 to R103, R98 to R104, R99 to R105, R100 to R106, R101 to R107, R102 to R108, R103 to R109, R104 to R110, R105 to R111, R106 to R112, R107 to R113, R108 to R114, R109 to R115, R110 to R116, R111 to R117, R112 to R118, R113 to R119, R114 to R120, R115 to R121, R125 to R122, R116 to R123, R117 to R124, R118 to R125, R119 to R126, R120 to R127, R121 to R128, R122 to R129, R123 to R130, R124 to R131, R93 to R99
Connections:
- net ~{CS}: now also R122.2
- net at R124.2, U19.18 (CS_{n}): no longer R122.2
Other:
- moved on the sheet: R122

Commit message: Different Matching Circuit
Parts:
- added C236, C237, C238: 100n, Capacitor_SMD:C_0402_1005Metric, symbol Device:C_Small
- added J34: SYNC, symbol Connector:Conn_Coaxial_Small
- added J35: REF, symbol Connector:Conn_Coaxial_Small
- added R230, R232, R235: 49.9, symbol Device:R_Small
- added R231, R236: 0, symbol Device:R_Small
- added R233, R234: 240, symbol Device:R_Small
Connections:
- net GND: now also C237.2, J34.2 (Ext), J35.2 (Ext), R230.2, R232.2, R233.2, R234.2, R235.2
- net at U19.37 (CLKIN0_{P}): now also C236.2
- net at U19.38 (CLKIN0_{N}): now also C237.1
- net at U19.6 (SYNC/SYSREFREQ): now also R236.2
- new net: C236.1, R231.2, R232.1, R234.1
- new net: J34.1 (In), R230.1, R236.1
- new net: C238.1, J35.1 (In), R235.1
- new net: C238.2, R231.1, R233.1
Other:
- moved on the sheet: C162, C163, R107, R108, R112, R116, R118, R120, R122, R124, R125, R126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
