File: lmk04828.kicad_sch (KiCad schematic)
At the start: 89 parts, among them J34 SYNC, J35 REF, U18 XX-XXX-VVXXFFF.fffff, U19 LMK0482x, Y2 ASE-xxxMHz

Commit message: For Darrel
Parts:
- renumbered C135 to C58, C136 to C59, C137 to C60, C138 to C61, C139 to C62, C140 to C63, C141 to C64, C142 to C65, C143 to C66, C144 to C67, C145 to C68, C146 to C69, C147 to C70, C148 to C71, C149 to C72, C150 to C73, C151 to C74, C152 to C75, C153 to C76, C154 to C77, C155 to C78, C156 to C79, C157 to C80, C238 to C81, C236 to C82, C237 to C83, C162 to C84, C163 to C85, C158 to C86, C159 to C87, C160 to C88, C161 to C89, C164 to C90, C165 to C91, C166 to C92, C167 to C93, C168 to C94, C169 to C95, J34 to J16, J35 to J17, R99 to R29, R100 to R30, R101 to R31, R102 to R32, R103 to R33, R104 to R34, R107 to R35, R108 to R36, R112 to R37, R105 to R38, R106 to R39, R230 to R40, R235 to R41, R236 to R42, R109 to R43, R110 to R44, R233 to R45, R116 to R46, R231 to R47, R118 to R48, R111 to R49, R234 to R50, R120 to R51, R113 to R52, R232 to R53, R114 to R54, R115 to R55, R117 to R56, R119 to R57, R121 to R58, R123 to R59, R122 to R60, R124 to R61, R125 to R62, R126 to R63, R127 to R64, R128 to R65, R129 to R66, R130 to R67, R131 to R68, R132 to R69, R133 to R70, R134 to R71, R135 to R72, TP8 to TP9, U18 to U12, U19 to U13

Commit message: wip
Parts:
- added R102, R104: 453k, Resistor_SMD:R_0402_1005Metric, symbol Device:R_Small
- added R103, R105: 33k, Resistor_SMD:R_0402_1005Metric, symbol Device:R_Small
Connections:
- net GND: now also R103.2, R105.2
- new net Linear POL LMK DIG/PGFB+: R102.1
- new net Linear POL LMK DIG/PGFB-: R102.2
- new net Linear POL LMK DIG/SET: R103.1
- new net Linear POL LMK VCO/PGFB+: R104.1
- new net Linear POL LMK VCO/PGFB-: R104.2
- new net Linear POL LMK VCO/SET: R105.1
- no-connect marks 2 -> 4
Other:
- added sheet Linear POL LMK DIG (linear.kicad_sch)
- added sheet Linear POL LMK VCO (linear.kicad_sch)

Commit message: Add Clock sources and monitor output
Parts:
- renumbered C93 to C100, C94 to C101, C95 to C102, C58 to C65, C59 to C66, C60 to C67, C61 to C68, C62 to C69, C63 to C70, C64 to C71, C65 to C72, C66 to C73, C67 to C74, C68 to C75, C69 to C76, C70 to C77, C71 to C78, C72 to C79, C73 to C80, C74 to C81, C75 to C82, C76 to C83, C77 to C84, C78 to C85, C79 to C86, C80 to C87, C81 to C88, C82 to C89, C83 to C90, C84 to C91, C85 to C92, C86 to C93, C87 to C94, C88 to C95, C89 to C96, C90 to C97, C91 to C98, C92 to C99, J16 to J24, J17 to J25, R29 to R28, R30 to R29, R31 to R30, R32 to R31, R33 to R32, R34 to R33, R35 to R34, R36 to R35, R37 to R36, R38 to R37, R39 to R38, R40 to R39, R41 to R40, R102 to R41, R103 to R42, R42 to R43, R43 to R44, R44 to R45, R45 to R46, R46 to R47, R47 to R48, R48 to R49, R49 to R50, R50 to R51, R51 to R52, R52 to R53, R53 to R54, R54 to R55, R55 to R56, R56 to R57, R57 to R58, R104 to R59, R105 to R60, R58 to R61, R59 to R62, R60 to R63, R61 to R64, R62 to R65, R63 to R66, R64 to R67, R65 to R68, R66 to R69, R67 to R70, R68 to R71, R69 to R72, R70 to R73, R71 to R74, R72 to R75, U12 to U18, U13 to U19, Y2 to Y3
Connections:
- net HF Out 4/C+: no longer names the net of U19.24 (DCLK4_{P})
- net HF Out 4/C-: no longer names the net of U19.25 (DCLK4_{N})
- net HF Out 5/C+: no longer names the net of U19.22 (SDCLK5_{P})
- net HF Out 5/C-: no longer names the net of U19.23 (SDCLK5_{N})
- net HF Out 6/C+: no longer names the net of U19.27 (DCLK6_{P})
- net HF Out 6/C-: no longer names the net of U19.28 (DCLK6_{N})
- net HF Out 7/C+: no longer names the net of U19.29 (SDCLK7_{P})
- net HF Out 7/C-: no longer names the net of U19.30 (SDCLK7_{N})
- net LF Balun Output 8/C+: no longer names the net of U19.51 (DCLK8_{P})
- net LF Balun Output 8/C-: no longer names the net of U19.52 (DCLK8_{N})
- no-connect marks 4 -> 14
Other:
- removed sheet HF Out 4
- removed sheet HF Out 5
- removed sheet HF Out 6
- removed sheet HF Out 7
- removed sheet LF Balun Output 8
- sheet LF Balun Output 10 ports: added OUT+, OUT-; removed none
- sheet LF Balun Output 11 ports: added OUT+, OUT-; removed none
- sheet LF Balun Output 9 ports: added OUT+, OUT-; removed none

Commit message: Round 1 review comments
Parts:
- added C105, C106, C107, C108: 100n, Capacitor_SMD:C_0402_1005Metric, symbol Device:C_Small
- added R102, R103, R106, R107: 240, symbol Device:R_Small
- renumbered C98 to C100, C99 to C101, C100 to C102, C101 to C103, C102 to C104, C65 to C67, C66 to C68, C67 to C69, C68 to C70, C69 to C71, C70 to C72, C71 to C73, C72 to C74, C73 to C75, C74 to C76, C75 to C77, C76 to C78, C77 to C79, C78 to C80, C79 to C81, C80 to C82, C81 to C83, C82 to C84, C83 to C85, C84 to C86, C85 to C87, C86 to C88, C87 to C89, C88 to C90, C89 to C91, C90 to C92, C91 to C93, C92 to C94, C93 to C95, C94 to C96, C95 to C97, C96 to C98, C97 to C99, J24 to J25, J25 to J26, R72 to R100, R73 to R101, R74 to R104, R75 to R105, R28 to R56, R29 to R57, R30 to R58, R31 to R59, R32 to R60, R33 to R61, R34 to R62, R35 to R63, R36 to R64, R37 to R65, R38 to R66, R39 to R67, R40 to R68, R41 to R69, R42 to R70, R43 to R71, R44 to R72, R45 to R73, R46 to R74, R47 to R75, R48 to R76, R49 to R77, R50 to R78, R51 to R79, R52 to R80, R53 to R81, R54 to R82, R55 to R83, R56 to R84, R57 to R85, R58 to R86, R59 to R87, R60 to R88, R61 to R89, R62 to R90, R63 to R91, R64 to R92, R65 to R93, R66 to R94, R67 to R95, R68 to R96, R69 to R97, R70 to R98, R71 to R99
Connections:
- net Linear POL LMK DIG/PGFB+ is gone; now on net +3.3VA_LMKDIG: R69.1
- net Linear POL LMK VCO/PGFB+ is gone; now on net +3.3VA_LMKCGVCO: R87.1
- net DCLK0n: no longer R100.1
- net DCLK0p: no longer R104.1
- net GND: now also R102.2, R103.2, R106.2, R107.2
- net HF Out 2/C+: now also U19.24 (DCLK4_{P}); no longer U19.15 (DCLK2_{P})
- net HF Out 2/C-: now also U19.25 (DCLK4_{N}); no longer U19.16 (DCLK2_{N})
- net HF Out 3/C+: now also U19.22 (SDCLK5_{P}); no longer U19.13 (SDCLK3_{P})
- net HF Out 3/C-: now also U19.23 (SDCLK5_{N}); no longer U19.14 (SDCLK3_{N})
- net SDCLK1n: no longer R101.1
- net SDCLK1p: no longer R105.1
- net at C103.1, U19.3 (SDCLK1_{P}): now also R105.1
- net at C104.1, U19.4 (SDCLK1_{N}): now also R101.1
- net at C101.1, U19.1 (DCLK0_{P}): now also R104.1
- net at C102.1, U19.2 (DCLK0_{N}): now also R100.1
- net Linear POL LMK DIG/PGFB- renamed Linear POL LMK DIG/PGFB
- net Linear POL LMK VCO/PGFB- renamed Linear POL LMK VCO/PGFB
- new net: C106.1, R102.1, U19.16 (DCLK2_{N})
- new net: C107.1, R107.1, U19.13 (SDCLK3_{P})
- new net: C108.1, R103.1, U19.14 (SDCLK3_{N})
- new net: C105.1, R106.1, U19.15 (DCLK2_{P})
- new net DCLK2n: C106.2
- new net DCLK2p: C105.2
- new net SDCLK3n: C108.2
- new net SDCLK3p: C107.2
- no-connect marks 14 -> 10
Other:
- sheet Linear POL LMK DIG ports: added PGFB; removed PGFB+, PGFB-
- sheet Linear POL LMK VCO ports: added PGFB; removed PGFB+, PGFB-
- moved on the sheet: C101, C102, C103, C104, R100, R101, R104, R105

Commit message: Round 2 Review, power tree cleanup
Parts:
- renumbered C98 to C100, C99 to C101, C100 to C102, C101 to C103, C102 to C104, C103 to C105, C104 to C106, C105 to C107, C106 to C108, C107 to C109, C108 to C110, C67 to C69, C68 to C70, C69 to C71, C70 to C72, C71 to C73, C72 to C74, C73 to C75, C74 to C76, C75 to C77, C76 to C78, C77 to C79, C78 to C80, C79 to C81, C80 to C82, C81 to C83, C82 to C84, C83 to C85, C84 to C86, C85 to C87, C86 to C88, C87 to C89, C88 to C90, C89 to C91, C90 to C92, C91 to C93, C92 to C94, C93 to C95, C94 to C96, C95 to C97, C96 to C98, C97 to C99, J25 to J26, J26 to J27, R90 to R100, R91 to R101, R92 to R102, R93 to R103, R94 to R104, R95 to R105, R96 to R106, R97 to R107, R98 to R108, R99 to R109, R100 to R110, R101 to R111, R102 to R112, R103 to R113, R104 to R114, R105 to R115, R106 to R116, R107 to R117, R56 to R66, R57 to R67, R58 to R68, R59 to R69, R60 to R70, R61 to R71, R62 to R72, R63 to R73, R64 to R74, R65 to R75, R66 to R76, R67 to R77, R68 to R78, R69 to R79, R70 to R80, R71 to R81, R72 to R82, R73 to R83, R74 to R84, R75 to R85, R76 to R86, R77 to R87, R78 to R88, R79 to R89, R80 to R90, R81 to R91, R82 to R92, R83 to R93, R84 to R94, R85 to R95, R86 to R96, R87 to R97, R88 to R98, R89 to R99
Connections:
- net CP: now also U19.32 (CP_{1}); no longer U19.46 (CP_{0})
- net at C100.1, C99.1: now also U19.46 (CP_{2}); no longer U19.32 (CP_{1})
