File: lmxmatchsingle.kicad_sch (KiCad schematic)
At the start: 9 parts

Commit message: Add mixer
Parts:
- renumbered C239 to C228, C240 to C229, C241 to C230, L13 to L11, R242 to R228, R243 to R229, R240 to R94, R241 to R95, TP10 to TP9
Changed lines of the file:
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@@
 		(on_board yes)
 		(dnp yes)
-		(property "Reference" "R242"
+		(property "Reference" "R228"
 			(at 115.57 116.8399 0)
 			(effects
@@
 					(unit 1)
 				)
+				(path "/eb9c972b-d134-41da-be97-ece3f463f7e0/d5a7e3c4-49dd-4cc7-9d82-7c02320e6daf/f37470a5-aa7e-4685-99e3-8b4186c25acc"
+					(reference "R228")
+					(unit 1)
+				)
 			)
 		)
@@
 		(on_board yes)
 		(dnp no)
-		(property "Reference" "#PWR0264"
+		(property "Reference" "#PWR0145"
 			(at 107.95 96.52 0)
 			(effects
@@
 				(path "/eb9c972b-d134-41da-be97-ece3f463f7e0/d5a7e3c4-49dd-4cc7-9d82-7c02320e6daf/e51e609f-c5bf-403c-8ca6-81342f1b9050"
 					(reference "#PWR0264")
+					(unit 1)
+				)
+				(path "/eb9c972b-d134-41da-be97-ece3f463f7e0/d5a7e3c4-49dd-4cc7-9d82-7c02320e6daf/f37470a5-aa7e-4685-99e3-8b4186c25acc"
+					(reference "#PWR0145")
 					(unit 1)
 				)
@@
 		(on_board yes)
 		(dnp no)
-		(property "Reference" "C239"
+		(property "Reference" "C228"
 			(at 123.19 100.584 90)
 			(effects
@@
 				(path "/eb9c972b-d134-41da-be97-ece3f463f7e0/d5a7e3c4-49dd-4cc7-9d82-7c02320e6daf/e51e609f-c5bf-403c-8ca6-81342f1b9050"
 					(reference "C239")
+					(unit 1)
+				)
+				(path "/eb9c972b-d134-41da-be97-ece3f463f7e0/d5a7e3c4-49dd-4cc7-9d82-7c02320e6daf/f37470a5-aa7e-4685-99e3-8b4186c25acc"
+					(reference "C228")
 					(unit 1)
 				)
@@
 		(on_board yes)
 		(dnp no)
-		(property "Reference" "C240"
+		(property "Reference" "C229"
 			(at 132.08 82.804 90)
 			(effects
@@
 					(unit 1)
 				)
+				(path "/eb9c972b-d134-41da-be97-ece3f463f7e0/d5a7e3c4-49dd-4cc7-9d82-7c02320e6daf/f37470a5-aa7e-4685-99e3-8b4186c25acc"
+					(reference "C229")
+					(unit 1)
+				)
 			)
 		)
@@
 		(dnp no)
 		(fields_autoplaced yes)
-		(property "Reference" "#PWR0267"
+		(property "Reference" "#PWR0244"
 			(at 161.29 104.14 0)
 			(effects
@@
 					(unit 1)
 				)
+				(path "/eb9c972b-d134-41da-be97-ece3f463f7e0/d5a7e3c4-49dd-4cc7-9d82-7c02320e6daf/f37470a5-aa7e-4685-99e3-8b4186c25acc"
+					(reference "#PWR0244")
+					(unit 1)
+				)
 			)
 		)
@@
 		(dnp no)
 		(fields_autoplaced yes)
-		(property "Reference" "#PWR0268"
+		(property "Reference" "#PWR0224"
 			(at 118.11 129.54 0)
 			(effects
@@
 					(unit 1)
 				)
+				(path "/eb9c972b-d134-41da-be97-ece3f463f7e0/d5a7e3c4-49dd-4cc7-9d82-7c02320e6daf/f37470a5-aa7e-4685-99e3-8b4186c25acc"
+					(reference "#PWR0224")
+					(unit 1)
+				)
 			)
 		)
@@
 		(on_board yes)
 		(dnp no)
-		(property "Reference" "R240"
+		(property "Reference" "R94"
 			(at 115.57 81.2799 0)
 			(effects
@@
 					(unit 1)
 				)
+				(path "/eb9c972b-d134-41da-be97-ece3f463f7e0/d5a7e3c4-49dd-4cc7-9d82-7c02320e6daf/f37470a5-aa7e-4685-99e3-8b4186c25acc"
+					(reference "R94")
+					(unit 1)
+				)
 			)
 		)
@@
 		(on_board yes)
 		(dnp no)
-		(property "Reference" "R241"
+		(property "Reference" "R95"
 			(at 115.57 106.6799 0)
 			(effects
@@
 					(unit 1)
 				)
+				(path "/eb9c972b-d134-41da-be97-ece3f463f7e0/d5a7e3c4-49dd-4cc7-9d82-7c02320e6daf/f37470a5-aa7e-4685-99e3-8b4186c25acc"
+					(reference "R95")
+					(unit 1)
+				)
 			)
 		)
@@
 		(on_board yes)
 		(dnp no)
-		(property "Reference" "R243"
+		(property "Reference" "R229"
 			(at 144.78 116.8399 0)
 			(effects
@@
 				(path "/eb9c972b-d134-41da-be97-ece3f463f7e0/d5a7e3c4-49dd-4cc7-9d82-7c02320e6daf/e51e609f-c5bf-403c-8ca6-81342f1b9050"
 					(reference "R243")
+					(unit 1)
+				)
+				(path "/eb9c972b-d134-41da-be97-ece3f463f7e0/d5a7e3c4-49dd-4cc7-9d82-7c02320e6daf/f37470a5-aa7e-4685-99e3-8b4186c25acc"
+					(reference "R229")
 					(unit 1)
 				)
@@
 		(on_board yes)
 		(dnp no)
-		(property "Reference" "C241"
+		(property "Reference" "C230"
 			(at 132.08 118.364 90)
 			(effects
@@
 					(unit 1)
 				)
+				(path "/eb9c972b-d134-41da-be97-ece3f463f7e0/d5a7e3c4-49dd-4cc7-9d82-7c02320e6daf/f37470a5-aa7e-4685-99e3-8b4186c25acc"
+					(reference "C230")
+					(unit 1)
+				)
 			)
 		)
@@
 		(dnp no)
 		(fields_autoplaced yes)
-		(property "Reference" "#PWR0265"
+		(property "Reference" "#PWR0229"
 			(at 128.27 104.14 0)
 			(effects
@@
 					(unit 1)
 				)
+				(path "/eb9c972b-d134-41da-be97-ece3f463f7e0/d5a7e3c4-49dd-4cc7-9d82-7c02320e6daf/f37470a5-aa7e-4685-99e3-8b4186c25acc"
+					(reference "#PWR0229")
+					(unit 1)
+				)
 			)
 		)
@@
 		(on_board yes)
 		(dnp no)
-		(property "Reference" "L13"
+		(property "Reference" "L11"
 			(at 113.03 89.916 90)
 			(effects
@@
 					(unit 1)
 				)
+				(path "/eb9c972b-d134-41da-be97-ece3f463f7e0/d5a7e3c4-49dd-4cc7-9d82-7c02320e6daf/f37470a5-aa7e-4685-99e3-8b4186c25acc"
+					(reference "L11")
+					(unit 1)
+				)
 			)
 		)
@@
 		(dnp no)
 		(fields_autoplaced yes)
-		(property "Reference" "#PWR0269"
+		(property "Reference" "#PWR0243"
 			(at 147.32 129.54 0)
 			(effects
@@
 					(unit 1)
 				)
+				(path "/eb9c972b-d134-41da-be97-ece3f463f7e0/d5a7e3c4-49dd-4cc7-9d82-7c02320e6daf/f37470a5-aa7e-4685-99e3-8b4186c25acc"
+					(reference "#PWR0243")
+					(unit 1)
+				)
 			)
 		)
@@
 		(on_board yes)
 		(dnp no)
-		(property "Reference" "TP10"
+		(property "Reference" "TP9"
 			(at 152.4 71.12 0)
 			(effects
@@
 					(unit 1)
 				)
+				(path "/eb9c972b-d134-41da-be97-ece3f463f7e0/d5a7e3c4-49dd-4cc7-9d82-7c02320e6daf/f37470a5-aa7e-4685-99e3-8b4186c25acc"
+					(reference "TP9")
+					(unit 1)
+				)
