File: rfpsu.kicad_sch (KiCad schematic)
At the start: 36 parts, among them J4 VSENSE, U4 LT8625S

Commit message: reorg and add 10MHz
Parts:
- renumbered R25 to R13, R26 to R14, R27 to R15, R28 to R16, R29 to R17, R30 to R18

Commit message: Renumber refdes
Parts:
- renumbered C34 to C48, C35 to C49, C36 to C50, C37 to C51, C38 to C52, C39 to C53, C40 to C54, C41 to C55, C42 to C56, C43 to C57, C44 to C58, C45 to C59, C46 to C60, C47 to C61, C48 to C62, C49 to C63, C50 to C64, C51 to C65, C52 to C66, C53 to C67, C54 to C68, J4 to J5, L3 to L4, L4 to L5, R13 to R21, R14 to R22, R15 to R23, R16 to R24, R17 to R25, R18 to R26, U4 to U6

Commit message: Add lmk and bump schematic size
Connections:
- net INTVCC: now reaches C55.1, TP2.1, U6.9 (INTVCC)
Changed lines of the file:
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@@
 	(generator "eeschema")
 	(generator_version "9.0")
-	(paper "A4")
+	(paper "A3")
 	(text "0.22uH 34A ISAT\nSRP7028AA-R22M"
 		(exclude_from_sim no)
@@
 		(effects
 			(font
+				(size 1.27 1.27)
+			)
+			(justify left)
+		)
+	)
+	(hierarchical_label "INTVCC"
+		(shape input)
+		(at 99.06 57.15 90)
+		(effects
+			(font
