File: rfpsu.kicad_sch (KiCad schematic)
At the start: 36 parts, among them J5 VSENSE, U6 LT8625S

Commit message: For Darrel
Parts:
- renumbered C48 to C21, C49 to C22, C50 to C23, C51 to C24, C52 to C25, C53 to C26, C54 to C27, C55 to C28, C56 to C29, C57 to C30, C58 to C31, C59 to C32, C60 to C33, C61 to C34, C62 to C35, C63 to C36, C64 to C37, C65 to C38, C66 to C39, C67 to C40, C68 to C41, J5 to J10, L4 to L3, L5 to L4, R21 to R11, R22 to R12, R23 to R13, R24 to R14, R25 to R15, R26 to R16, TP2 to TP3, TP3 to TP4, TP4 to TP5, TP5 to TP6, TP6 to TP7, U6 to U7

Commit message: Add Clock sources and monitor output
Parts:
- renumbered C21 to C11, C22 to C12, C23 to C13, C24 to C14, C25 to C15, C26 to C16, C27 to C17, C28 to C18, C29 to C19, C30 to C20, C31 to C21, C32 to C22, C33 to C23, C34 to C24, C35 to C25, C36 to C26, C37 to C27, C38 to C28, C39 to C29, C40 to C30, C41 to C31, J10 to J17, L3 to L2, L4 to L3, R12 to R10, R13 to R11, R14 to R12, R15 to R13, R16 to R14, R11 to R9, U7 to U10
