File: rfpsu.kicad_sch (KiCad schematic)
At the start: 36 parts, among them J17 VSENSE, U10 LT8625S

Commit message: Round 1 review comments
Parts:
- removed R13: 10, Resistor_SMD:R_0402_1005Metric, symbol Device:R_Small
- added C? (x2): DNP, Capacitor_SMD:C_0402_1005Metric, symbol Device:C_Small
- C33: renamed from C31; value 470p -> 1n; DIGIKEY_PN 490-GCM155R71H471KA37JCT-ND -> (none)
- renumbered C11 to C13, C12 to C14, C13 to C15, C14 to C16, C15 to C17, C16 to C18, C17 to C19, C18 to C20, C19 to C21, C20 to C22, C21 to C23, C22 to C24, C23 to C25, C24 to C26, C25 to C27, C26 to C28, C27 to C29, C28 to C30, C29 to C31, C30 to C32, R9 to R12, R10 to R13, R11 to R14, R12 to R15, R14 to R17
Connections:
- net GND: now also C?.1
- net PGFB+: now also C?.2
- net OUTS: now reaches U10.13 (OUTS)
- net OUTS: now also C?.1, C?.2

Commit message: Round 2 Review, power tree cleanup
Parts:
- gave numbers to parts that had none: 2
- renumbered C33 to C35, J17 to J18, R12 to R14, R13 to R15, R14 to R16, R15 to R17, R17 to R18

Commit message: Darrel Suggestions
Parts:
- renumbered L2 to L1, L3 to L2

Commit message: add NC and fix ERC
Parts:
- removed C25: 1u, Capacitor_SMD:C_0402_1005Metric, symbol Device:C_Small
Connections:
- net VIN: now also U10.23 (NC)
- net at L1.1, TP7.1, U10.1 (SW)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: now also U10.22 (NC)
- net PGFB+ renamed VOUT
- new net: U10.24 (NC), U10.25 (NC)
- no-connect marks 0 -> 2
Changed lines of the file:
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@@
 	)
 	(junction
-		(at 241.3 43.18)
-		(diameter 0)
-		(color 0 0 0 0)
-	)
-	(junction
 		(at 46.99 33.02)
 		(diameter 0)
@@
 		(color 0 0 0 0)
 	)
+	(no_connect
+		(at 158.75 35.56)
+	)
+	(no_connect
+		(at 158.75 67.31)
+	)
 	(wire
 		(pts
@@
 	(wire
 		(pts
-			(xy 161.29 41.91) (xy 161.29 43.18)
-		)
-		(stroke
-			(width 0)
-			(type default)
-		)
-	)
-	(wire
-		(pts
 			(xy 29.21 43.18) (xy 29.21 45.72)
 		)
@@
 	(wire
 		(pts
-			(xy 236.22 43.18) (xy 241.3 43.18)
+			(xy 236.22 43.18) (xy 262.89 43.18)
 		)
 		(stroke
@@
 	(wire
 		(pts
-			(xy 241.3 43.18) (xy 241.3 45.72)
-		)
-		(stroke
-			(width 0)
-			(type default)
-		)
-	)
-	(wire
-		(pts
 			(xy 29.21 33.02) (xy 38.1 33.02)
 		)
@@
 	(wire
 		(pts
-			(xy 158.75 35.56) (xy 161.29 35.56)
-		)
-		(stroke
-			(width 0)
-			(type default)
-		)
-	)
-	(wire
-		(pts
 			(xy 90.17 73.66) (xy 90.17 76.2)
 		)
@@
 	(wire
 		(pts
-			(xy 241.3 43.18) (xy 262.89 43.18)
-		)
-		(stroke
-			(width 0)
-			(type default)
-		)
-	)
-	(wire
-		(pts
 			(xy 236.22 22.86) (xy 241.3 22.86)
 		)
@@
 	(wire
 		(pts
-			(xy 161.29 35.56) (xy 161.29 36.83)
-		)
-		(stroke
-			(width 0)
-			(type default)
-		)
-	)
-	(wire
-		(pts
 			(xy 29.21 33.02) (xy 29.21 35.56)
 		)
@@
 		)
 	)
-	(hierarchical_label "PGFB+"
-		(shape input)
-		(at 241.3 45.72 0)
-		(effects
-			(font
-				(size 1.27 1.27)
-			)
-			(justify left)
-		)
-	)
 	(hierarchical_label "PGFB-"
 		(shape input)
@@
 	)
 	(symbol
+		(lib_id "power:PWR_FLAG")
+		(at 262.89 43.18 270)
+		(unit 1)
+		(body_style 1)
+		(exclude_from_sim no)
+		(in_bom yes)
+		(on_board yes)
+		(in_pos_files yes)
+		(dnp no)
+		(fields_autoplaced yes)
+		(property "Reference" "#FLG014"
+			(at 264.795 43.18 0)
+			(hide yes)
+			(show_name no)
+			(do_not_autoplace no)
+			(effects
+				(font
+					(size 1.27 1.27)
+				)
+			)
+		)
+		(property "Value" "PWR_FLAG"
+			(at 266.7 43.1799 90)
+			(show_name no)
+			(do_not_autoplace no)
+			(effects
+				(font
+					(size 1.27 1.27)
+				)
+				(justify left)
+			)
+		)
+		(property "Footprint" ""
+			(at 262.89 43.18 0)
+			(hide yes)
+			(show_name no)
+			(do_not_autoplace no)
+			(effects
+				(font
+					(size 1.27 1.27)
+				)
+			)
+		)
+		(property "Datasheet" ""
+			(at 262.89 43.18 0)
+			(hide yes)
+			(show_name no)
+			(do_not_autoplace no)
+			(effects
+				(font
+					(size 1.27 1.27)
+				)
+			)
+		)
+		(property "Description" "Special symbol for telling ERC where power comes from"
+			(at 262.89 43.18 0)
+			(hide yes)
+			(show_name no)
+			(do_not_autoplace no)
+			(effects
+				(font
+					(size 1.27 1.27)
+				)
+			)
+		)
+		(pin "1"
+		)
+		(instances
+			(project "huskypointofload"
+				(path "/eb9c972b-d134-41da-be97-ece3f463f7e0/28dccbc8-62a2-4750-b12f-4e220cef19bd/1f40507f-5f9f-444c-b99e-42dfd163ee6e"
+					(reference "#FLG015")
+					(unit 1)
+				)
+				(path "/eb9c972b-d134-41da-be97-ece3f463f7e0/28dccbc8-62a2-4750-b12f-4e220cef19bd/f8e9761d-04af-4a91-85c5-fba55f506320"
+					(reference "#FLG014")
+					(unit 1)
+				)
+				(path "/eb9c972b-d134-41da-be97-ece3f463f7e0/e3b9a158-a3aa-4eeb-b09d-59c46f782af5/ff11547f-04ea-462c-b501-e564f5dcf459"
+					(reference "#FLG016")
+					(unit 1)
+				)
+			)
+		)
+	)
+	(symbol
 		(lib_id "Device:C_Small")
 		(at 107.95 71.12 0)
@@
 	)
 	(symbol
-		(lib_id "Device:C_Small")
-		(at 161.29 39.37 0)
-		(unit 1)
-		(body_style 1)
-		(exclude_from_sim no)
-		(in_bom yes)
-		(on_board yes)
-		(in_pos_files yes)
-		(dnp no)
-		(property "Reference" "C25"
-			(at 163.83 38.1062 0)
-			(show_name no)
-			(do_not_autoplace no)
-			(effects
-				(font
-					(size 1.27 1.27)
-				)
-				(justify left)
-			)
-		)
-		(property "Value" "1u"
-			(at 163.83 40.6462 0)
-			(show_name no)
-			(do_not_autoplace no)
-			(effects
-				(font
-					(size 1.27 1.27)
-				)
-				(justify left)
-			)
-		)
-		(property "Footprint" "Capacitor_SMD:C_0402_1005Metric"
-			(at 161.29 39.37 0)
-			(hide yes)
-			(show_name no)
-			(do_not_autoplace no)
-			(effects
-				(font
-					(size 1.27 1.27)
-				)
-			)
-		)
-		(property "Datasheet" ""
-			(at 161.29 39.37 0)
-			(hide yes)
-			(show_name no)
-			(do_not_autoplace no)
-			(effects
-				(font
-					(size 1.27 1.27)
-				)
-			)
-		)
-		(property "Description" "Unpolarized capacitor, small symbol"
-			(at 161.29 39.37 0)
-			(hide yes)
-			(show_name no)
-			(do_not_autoplace no)
-			(effects
-				(font
-					(size 1.27 1.27)
-				)
-			)
-		)
-		(property "DIGIKEY_PN" "490-14409-1-ND"
-			(at 161.29 39.37 0)
-			(hide yes)
-			(show_name no)
-			(do_not_autoplace no)
-			(effects
-				(font
-					(size 1.27 1.27)
-				)
-			)
-		)
-		(pin "2"
-		)
-		(pin "1"
-		)
-		(instances
-			(project "huskypointofload"
-				(path "/eb9c972b-d134-41da-be97-ece3f463f7e0/28dccbc8-62a2-4750-b12f-4e220cef19bd/1f40507f-5f9f-444c-b99e-42dfd163ee6e"
-					(reference "C259")
-					(unit 1)
-				)
-				(path "/eb9c972b-d134-41da-be97-ece3f463f7e0/28dccbc8-62a2-4750-b12f-4e220cef19bd/f8e9761d-04af-4a91-85c5-fba55f506320"
-					(reference "C25")
-					(unit 1)
-				)
-				(path "/eb9c972b-d134-41da-be97-ece3f463f7e0/e3b9a158-a3aa-4eeb-b09d-59c46f782af5/ff11547f-04ea-462c-b501-e564f5dcf459"
-					(reference "C294")
-					(unit 1)
-				)
-			)
-		)
-	)
-	(symbol
 		(lib_id "huskylib:LT8625S")
 		(at 143.51 46.99 0)
@@
 		(pin "14"
 		)
+		(pin "22"
+		)
+		(pin "23"
+		)
+		(pin "24"
+		)
+		(pin "25"
+		)
 		(instances
