File: bias_gen.kicad_sch (KiCad schematic)
At the start: 37 parts, among them U18 ADA4522-4, U19 AD5696R

Commit message: For Darrel
Parts:
- renumbered C148 to C130, C149 to C131, C152 to C132, C153 to C133, C154 to C134, C155 to C135, C156 to C136, C157 to C137, C151 to C138, C150 to C139, C158 to C140, C159 to C141, C160 to C142, C161 to C143, R117 to R152, R102 to R153, R103 to R154, R105 to R155, R106 to R156, R104 to R157, R107 to R158, R101 to R159, R108 to R160, R113 to R161, R114 to R162, R109 to R163, R110 to R164, R115 to R165, R111 to R166, R116 to R167, R112 to R168, U19 to U17
