File: linear.kicad_sch (KiCad schematic)
At the start: 8 parts, among them J3 VSENSE, U2 LT3045xDD

Commit message: For Darrel
Parts:
- renumbered C28 to C1, C29 to C2, C30 to C3, J3 to J8, R13 to R3, R14 to R4, R15 to R5, U2 to U3
