File: linear.kicad_sch (KiCad schematic)
At the start: 8 parts, among them J8 VSENSE, U3 LT3045xDD

Commit message: wip
Parts:
- renumbered C1 to C114, C2 to C115, C3 to C116, J8 to J25, R3 to R135, R4 to R136, R5 to R137, U3 to U15

Commit message: Add Clock sources and monitor output
Parts:
- renumbered C114 to C1, C115 to C2, C116 to C3, J25 to J15, R135 to R3, R136 to R4, R137 to R5, U15 to U3

Commit message: Round 1 review comments
Parts:
- added C2: 4.7u, symbol Device:C_Small
- renumbered C2 to C3, C3 to C4, R3 to R6, R4 to R7, R5 to R8
Connections:
- net PGFB- is gone; now on net PGFB: R8.1
- net GND: now also C2.2
- net SET: now also C2.1
- net PGFB+ renamed PGFB

Commit message: Round 2 Review, power tree cleanup
Parts:
- renumbered J15 to J16, R8 to R10, R6 to R8, R7 to R9

Commit message: Passive footprint pass
Parts:
- C2: footprint (none) -> Capacitor_SMD:C_0402_1005Metric
Changed lines of the file:
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@@
 			)
 		)
-		(property "Footprint" ""
+		(property "Footprint" "Capacitor_SMD:C_0402_1005Metric"
 			(at 107.95 102.87 0)
 			(hide yes)
