File: linear.kicad_sch (KiCad schematic)
At the start: 9 parts, among them J16 VSENSE, U3 LT3045xDD

Commit message: add NC and fix ERC
Parts:
- removed C2: 4.7u, Capacitor_SMD:C_0402_1005Metric, symbol Device:C_Small
- added C2: 4.7u, Capacitor_Tantalum_SMD:CP_EIA-2012-15_AVX-P, symbol Device:C_Polarized_Small
Connections:
- net GND: now also C2.2
- net SET: now also C2.1
Changed lines of the file:
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@@
-	)
-	(junction
-		(at 95.25 109.22)
-		(diameter 0)
-		(color 0 0 0 0)
 	)
 	(junction
@@
 		(pts
 			(xy 129.54 109.22) (xy 139.7 109.22)
-		)
-		(stroke
-			(width 0)
-			(type default)
-		)
-	)
-	(wire
-		(pts
-			(xy 83.82 104.14) (xy 83.82 109.22)
-		)
-		(stroke
-			(width 0)
-			(type default)
-		)
-	)
-	(wire
-		(pts
-			(xy 83.82 109.22) (xy 95.25 109.22)
 		)
 		(stroke
@@
 			)
 			(justify left)
-		)
-	)
-	(hierarchical_label "ILIM-"
-		(shape input)
-		(at 83.82 104.14 180)
-		(effects
-			(font
-				(size 1.27 1.27)
-			)
-			(justify right)
 		)
 	)
@@
 	)
 	(symbol
-		(lib_name "C_Small_1")
-		(lib_id "Device:C_Small")
+		(lib_id "Device:C_Polarized_Small")
 		(at 107.95 102.87 0)
 		(unit 1)
@@
 		(fields_autoplaced yes)
 		(property "Reference" "C2"
-			(at 110.49 101.5999 0)
+			(at 110.49 101.0538 0)
 			(show_name no)
 			(do_not_autoplace no)
@@
 		)
 		(property "Value" "4.7u"
-			(at 110.49 104.1399 0)
+			(at 110.49 103.5938 0)
 			(show_name no)
 			(do_not_autoplace no)
@@
 			)
 		)
-		(property "Footprint" "Capacitor_SMD:C_0402_1005Metric"
+		(property "Footprint" "Capacitor_Tantalum_SMD:CP_EIA-2012-15_AVX-P"
 			(at 107.95 102.87 0)
 			(hide yes)
@@
 			)
 		)
-		(property "Datasheet" ""
+		(property "Datasheet" "https://www.vishay.com/docs/40179/tmcp.pdf"
 			(at 107.95 102.87 0)
 			(hide yes)
@@
 			)
 		)
-		(property "Description" "Unpolarized capacitor, small symbol"
-			(at 107.95 113.03 0)
-			(hide yes)
-			(show_name no)
+		(property "Description" "Polarized capacitor, small symbol"
+			(at 107.95 102.87 0)
+			(hide yes)
+			(show_name no)
+			(do_not_autoplace no)
+			(effects
+				(font
+					(size 1.27 1.27)
+				)
+			)
+		)
+		(property "DIGIKEY_PN" "718-TMCP1A475KTRFCT-ND"
+			(at 107.95 102.87 0)
+			(hide yes)
+			(show_name no)
