File: rf_supplies.kicad_sch (KiCad schematic)
At the start: 35 parts, among them J13 VSENSE, U15 INA290A2xDCK, U16 INA290A2xDCK

Commit message: For Darrel
Parts:
- removed C127, C129: 100n, Capacitor_SMD:C_0402_1005Metric, symbol Device:C_Small
- removed D9: DFLS1150, Diode_SMD:D_PowerDI-123, symbol Device:D_Schottky_Small
- removed F1: 10A, Fuse:Fuseholder_Littelfuse_Nano2_157x, symbol Device:Fuse
- removed R76: 5m, Resistor_SMD:R_2512_6332Metric, symbol Device:R
- removed R84: 1.5M, symbol Device:R_Small
- removed R85: 100k, Resistor_SMD:R_0402_1005Metric, symbol Device:R_Small
- removed U15: INA290A2xDCK, Package_TO_SOT_SMD:SOT-353_SC-70-5, symbol Amplifier_Current:INA290A2xDCK
- renumbered C126 to C102, C128 to C103, C130 to C104, C131 to C105, D10 to D11, F2 to F1, J13 to J20, L10 to L6, R88 to R100, R89 to R101, R86 to R102, R87 to R103, R90 to R104, R91 to R105, R92 to R106, R93 to R107, R244 to R108, R245 to R109, R77 to R93, R78 to R94, R79 to R95, R80 to R96, R81 to R97, R82 to R98, R83 to R99, U16 to U14
Other:
- removed sheet Linear POL Dist
- note removed: "Locate bead in IBC can"
