File: splitrail.kicad_sch (KiCad schematic)
At the start: 14 parts, among them U29 LTC3260xMSE

Commit message: For Darrel
Parts:
- renumbered C142 to C121, C143 to C122, C141 to C123, C135 to C124, C136 to C125, C137 to C126, C138 to C127, C139 to C128, C140 to C129, R99 to R148, R94 to R149, R95 to R150, R100 to R151, U29 to U16
