File: clocking.kicad_sch (KiCad schematic)
At the start: 10 parts, among them J37 RAMPCTL, J38 LOCTL, Q1 DTC143Z

Commit message: For Darrel
Parts:
- renumbered D11 to D10, D13 to D8, D12 to D9, J38 to J14, J37 to J15, R238 to R25, R237 to R26, R220 to R27, R239 to R28
