File: hmc525.kicad_sch (KiCad schematic)
At the start: 4 parts, among them U24 HMC525ALC4, U26 PAT1220-C-6DB

Commit message: For Darrel
Parts:
- renumbered TP16 to TP1, TP17 to TP2, U26 to U1, U24 to U2
Other:
- note added: "TODO: Power Locally"

Commit message: wip
Other:
- note removed: "TODO: Power Locally"
Changed lines of the file:
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@@
 	(generator_version "10.0")
 	(paper "A3")
-	(text "TODO: Power Locally"
-		(exclude_from_sim no)
-		(at 55.118 161.29 0)
-		(effects
-			(font
-				(size 1.27 1.27)
-			)
-		)
-	)
 	(junction
 		(at 148.59 167.64)
