File: MCU.kicad_sch (KiCad schematic)
At the start: 34 parts, among them J6 RS485, J7 JTAG, J8 USB-C, SW1 SYS_RESET, SW2 BOOT0, U7 STM32G474MBTx, U8 LTC2851xS8, U9 USBLC6-2SC6, Y1 16MHz

Commit message: For Darrel
Parts:
- renumbered C69 to C42, C70 to C43, C71 to C44, C72 to C45, C73 to C46, C74 to C47, C75 to C48, C76 to C49, C77 to C50, C78 to C51, C79 to C52, C80 to C53, D5 to D4, D6 to D5, D7 to D6, D8 to D7, J6 to J11, J7 to J12, J8 to J13, R27 to R17, R28 to R18, R29 to R19, R30 to R20, R31 to R21, R32 to R22, R33 to R23, R34 to R24, TP7 to TP8, U9 to U10, U7 to U8, U8 to U9
Connections:
- net BUCKIN_SENSE: no longer names the net of D5.2 (A), U8.13 (PA1)
- net BUCKOUT_SENSE: no longer names the net of D7.2 (A), U8.17 (PA3)
- net EN_IBC: no longer names the net of U8.69 (PD0)
- net HS_SWITCH: no longer names the net of U8.43 (PB12)
- net LS_SWITCH: no longer names the net of U8.44 (PB13)
- net MISO renamed CIPO
- net MOSI renamed COPI
- net SOC_ISENSE: no longer names the net of U8.8 (PC0)

Commit message: wip
Connections:
- net SEL0: no longer U8.75 (PB6)
- net SEL1: no longer U8.76 (PB7)
Changed lines of the file:
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@@
 	(wire
 		(pts
-			(xy 90.17 97.79) (xy 95.25 97.79)
+			(xy -6.35 88.9) (xy -1.27 88.9)
 		)
 		(stroke
@@
 	(wire
 		(pts
-			(xy 90.17 95.25) (xy 95.25 95.25)
+			(xy -6.35 86.36) (xy -1.27 86.36)
 		)
 		(stroke
@@
 	(hierarchical_label "SEL1"
 		(shape input)
-		(at 95.25 97.79 0)
+		(at -1.27 88.9 0)
 		(effects
 			(font
@@
 	(hierarchical_label "SEL0"
 		(shape input)
-		(at 95.25 95.25 0)
-		(effects
-			(font
+		(at -1.27 86.36 0)
+		(effects
+			(font

Commit message: wip
Parts:
- added U?: RP2354A, Package_DFN_QFN:QFN-60-1EP_7x7mm_P0.4mm_EP3.4x3.4mm, symbol MCU_RaspberryPi:RP2354A
Connections:
- new net: U?.1 (IOVDD), U?.11 (IOVDD), U?.20 (IOVDD), U?.30 (IOVDD), U?.38 (IOVDD), U?.45 (IOVDD)
- new net: U?.23 (DVDD), U?.39 (DVDD), U?.6 (DVDD)
Changed lines of the file:
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@@
+	)
+	(symbol
+		(lib_id "MCU_RaspberryPi:RP2354A")
+		(at 133.35 218.44 0)
+		(unit 1)
+		(body_style 1)
+		(exclude_from_sim no)
+		(in_bom yes)
+		(on_board yes)
+		(in_pos_files yes)
+		(dnp no)
+		(fields_autoplaced yes)
+		(property "Reference" "U?"
+			(at 135.4933 262.89 0)
+			(show_name no)
+			(do_not_autoplace no)
+			(effects
+				(font
+					(size 1.27 1.27)
+				)
+				(justify left)
+			)
+		)
+		(property "Value" "RP2354A"
+			(at 135.4933 265.43 0)
+			(show_name no)
+			(do_not_autoplace no)
+			(effects
+				(font
+					(size 1.27 1.27)
+				)
+				(justify left)
+			)
+		)
+		(property "Footprint" "Package_DFN_QFN:QFN-60-1EP_7x7mm_P0.4mm_EP3.4x3.4mm"
+			(at 133.35 218.44 0)
+			(hide yes)
+			(show_name no)
+			(do_not_autoplace no)
+			(effects
+				(font
+					(size 1.27 1.27)
+				)
+			)
+		)
+		(property "Datasheet" "https://datasheets.raspberrypi.com/rp2350/rp2350-datasheet.pdf"
+			(at 133.35 218.44 0)
+			(hide yes)
+			(show_name no)
+			(do_not_autoplace no)
+			(effects
+				(font
+					(size 1.27 1.27)
+				)
+			)
+		)
+		(property "Description" "A microcontroller by Raspberry Pi, dual CPU architecture (ARM Cortex-M33 / RISC-V Hazard3), 150MHz, 2MB flash, 520KB SRAM, 12 PIO state machines, VQFN-60"
+			(at 133.35 218.44 0)
+			(hide yes)
+			(show_name no)
+			(do_not_autoplace no)
+			(effects
+				(font
+					(size 1.27 1.27)
+				)
+			)
+		)
+		(property private "KLC_S4.2_DVDD" "Not a standalone power converter; internal on-chip voltage regulator for digital core supply; DVDD is the digital core power supply, should be placed next to voltage regulator output."
+			(at 133.35 220.98 0)
+			(hide yes)
+			(show_name yes)
+			(do_not_autoplace no)
+			(effects
+				(font
+					(size 1.27 1.27)
+				)
+			)
+		)
+		(property private "KLC_S4.2_VREG_LX" "Should be placed next to DVDD."
+			(at 133.35 220.98 0)
+			(hide yes)
+			(show_name yes)
+			(do_not_autoplace no)
+			(effects
+				(font
+					(size 1.27 1.27)
+				)
+			)
+		)
+		(pin "6"
+		)
+		(pin "36"
+		)
+		(pin "37"
+		)
+		(pin "38"
+		)
+		(pin "40"
+		)
+		(pin "41"
+		)
+		(pin "42"
+		)
+		(pin "43"
+		)
+		(pin "44"
+		)
+		(pin "45"
+		)
+		(pin "48"
+		)
+		(pin "49"
+		)
+		(pin "50"
+		)
+		(pin "51"
+		)
+		(pin "52"
+		)
+		(pin "55"
+		)
+		(pin "12"
+		)
+		(pin "13"
+		)
+		(pin "14"
+		)
+		(pin "56"
+		)
+		(pin "57"
+		)
+		(pin "58"
+		)
+		(pin "59"
+		)
+		(pin "60"
+		)
+		(pin "61"
+		)
+		(pin "39"
+		)
+		(pin "46"
+		)
+		(pin "47"
+		)
+		(pin "53"
+		)
+		(pin "54"
+		)
+		(pin "1"
+		)
+		(pin "2"
+		)
+		(pin "3"
+		)
+		(pin "4"
+		)
+		(pin "5"
+		)
+		(pin "7"
+		)
+		(pin "8"
+		)
+		(pin "9"
+		)
+		(pin "10"
+		)
+		(pin "11"
+		)
+		(pin "15"
+		)
+		(pin "16"
+		)
+		(pin "17"
+		)
+		(pin "18"
+		)
+		(pin "19"
+		)
+		(pin "20"
+		)
+		(pin "21"
+		)
+		(pin "22"
+		)
+		(pin "23"
+		)
+		(pin "24"
+		)
+		(pin "25"
+		)
+		(pin "26"
+		)
+		(pin "27"
+		)
+		(pin "28"
+		)
+		(pin "29"
+		)
+		(pin "30"
+		)
+		(pin "31"
+		)
+		(pin "32"
+		)
+		(pin "33"
+		)
+		(pin "34"
+		)
+		(pin "35"
+		)
+		(instances
+			(project "huskypointofload"
+				(path "/eb9c972b-d134-41da-be97-ece3f463f7e0/aad3f0e3-dcbe-4112-94dc-37caa60c9eb1"
+					(reference "U?")
+					(unit 1)
+				)
+			)
+		)
 	)
 	(symbol
