File: lmx2594.kicad_sch (KiCad schematic)
At the start: 46 parts, among them J32 TUNESENSE, J36 SYSREFREQ, U21 LMX2594

Commit message: For Darrel
Parts:
- renumbered C197 to C154, C198 to C155, C199 to C156, C208 to C157, C200 to C158, C201 to C159, C202 to C160, C210 to C161, C212 to C162, C213 to C163, C214 to C164, C216 to C165, C203 to C166, C217 to C167, C204 to C168, C219 to C169, C205 to C170, C220 to C171, C206 to C172, C207 to C173, C209 to C174, C211 to C175, C215 to C176, C218 to C177, C221 to C178, C222 to C179, C223 to C180, C224 to C181, J32 to J37, R209 to R184, R210 to R185, R219 to R186, R211 to R187, R212 to R188, R213 to R189, R214 to R190, R215 to R191, R216 to R192, R217 to R193, R218 to R194, R221 to R195, R222 to R196, R223 to R197, R224 to R198, U21 to U22

Commit message: wip
Parts:
- added R100, R106: 453k, Resistor_SMD:R_0402_1005Metric, symbol Device:R_Small
- added R101, R107: 33k, Resistor_SMD:R_0402_1005Metric, symbol Device:R_Small
Connections:
- net GND: now also R101.2, R107.2
- new net Linear POL LMX BUF/PGFB+: R106.1
- new net Linear POL LMX BUF/PGFB-: R106.2
- new net Linear POL LMX BUF/SET: R107.1
- new net Linear POL LMX/PGFB+: R100.1
- new net Linear POL LMX/PGFB-: R100.2
- new net Linear POL LMX/SET: R101.1
- no-connect marks 0 -> 2
Other:
- added sheet Linear POL LMX (linear.kicad_sch)
- added sheet Linear POL LMX BUF (linear.kicad_sch)
- moved on the sheet: C154, C155, C156, C158, C159, C160, C166, C168, C170, C172, C173, C174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

Commit message: Add Clock sources and monitor output
Parts:
- renumbered C157 to C144, C161 to C145, C154 to C146, C162 to C147, C163 to C148, C164 to C149, C155 to C150, C165 to C151, C156 to C152, C167 to C153, C169 to C154, C158 to C155, C159 to C156, C160 to C157, C171 to C158, C166 to C159, C168 to C160, C170 to C161, C172 to C162, C173 to C163, C178 to C164, C179 to C165, C180 to C166, C174 to C167, C181 to C168, C175 to C169, C176 to C170, C177 to C171, J36 to J34, J37 to J35, R100 to R151, R101 to R152, R184 to R153, R185 to R154, R186 to R155, R187 to R156, R188 to R157, R189 to R158, R190 to R159, R191 to R160, R192 to R161, R193 to R162, R194 to R163, R195 to R164, R196 to R165, R197 to R166, R106 to R167, R107 to R168, R198 to R169, U22 to U30

Commit message: Round 1 review comments
Parts:
- renumbered C144 to C109, C145 to C110, C146 to C111, C147 to C112, C148 to C113, C149 to C114, C150 to C115, C151 to C116, C152 to C117, C153 to C118, C154 to C119, C155 to C120, C156 to C121, C157 to C122, C158 to C123, C159 to C124, C160 to C125, C161 to C126, C162 to C127, C163 to C128, C164 to C129, C165 to C130, C166 to C131, C167 to C132, C168 to C133, C169 to C134, C170 to C135, C171 to C136, J34 to J27, J35 to J28, R151 to R108, R152 to R109, R153 to R110, R154 to R111, R155 to R112, R156 to R113, R157 to R114, R158 to R115, R159 to R116, R160 to R117, R161 to R118, R162 to R119, R163 to R120, R164 to R121, R165 to R122, R166 to R123, R167 to R124, R168 to R125, R169 to R126, U30 to U20
Connections:
- net Linear POL LMX BUF/PGFB+ is gone; now on net +3.3VA_LMXBUF: R124.1
- net Linear POL LMX/PGFB+ is gone; now on net +3.3VA_LMX: R108.1
- net Linear POL LMX BUF/PGFB- renamed Linear POL LMX BUF/PGFB
- net Linear POL LMX/PGFB- renamed Linear POL LMX/PGFB
Other:
- sheet Linear POL LMX ports: added PGFB; removed PGFB+, PGFB-
- sheet Linear POL LMX BUF ports: added PGFB; removed PGFB+, PGFB-
- moved on the sheet: C112, C113, R110

Commit message: Round 2 Review, power tree cleanup
Parts:
- renumbered C112 to C111, C113 to C112, C109 to C113, C110 to C114, C111 to C115, C114 to C116, C115 to C117, C116 to C118, C117 to C119, C118 to C120, C119 to C121, C120 to C122, C121 to C123, C122 to C124, C123 to C125, C124 to C126, C125 to C127, C126 to C128, C127 to C129, C128 to C130, C129 to C131, C130 to C132, C131 to C133, C132 to C134, C133 to C135, C134 to C136, C135 to C137, C136 to C138, J27 to J28, J28 to J29, R110 to R118, R108 to R119, R109 to R120, R111 to R121, R112 to R122, R113 to R123, R114 to R124, R115 to R125, R116 to R126, R117 to R127, R118 to R128, R119 to R129, R120 to R130, R121 to R131, R122 to R132, R123 to R133, R124 to R134, R125 to R135, R126 to R136

Commit message: Darrel Suggestions
Parts:
- C122, C123, C124, C129, C130, C138: value 100n -> 1u; DIGIKEY_PN 490-6969-1-ND -> 490-13394-1-ND

Commit message: Passive footprint pass
Parts:
- C113, C114, C116, C118, C119, C120, C121, C125, C128, C137: footprint (none) -> Capacitor_SMD:C_0402_1005Metric
- R118, R122: footprint (none) -> Resistor_SMD:R_0402_1005Metric
Changed lines of the file:
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@@
 			)
 		)
-		(property "Footprint" ""
+		(property "Footprint" "Capacitor_SMD:C_0402_1005Metric"
 			(at 69.85 144.78 0)
 			(hide yes)
@@
 			)
 		)
-		(property "Footprint" ""
+		(property "Footprint" "Capacitor_SMD:C_0402_1005Metric"
 			(at 80.01 144.78 0)
 			(hide yes)
@@
 			)
 		)
-		(property "Footprint" ""
+		(property "Footprint" "Capacitor_SMD:C_0402_1005Metric"
 			(at 59.69 144.78 0)
 			(hide yes)
@@
 			)
 		)
-		(property "Footprint" ""
+		(property "Footprint" "Capacitor_SMD:C_0402_1005Metric"
 			(at 90.17 144.78 0)
 			(hide yes)
@@
 			)
 		)
-		(property "Footprint" ""
+		(property "Footprint" "Capacitor_SMD:C_0402_1005Metric"
 			(at 110.49 144.78 0)
 			(hide yes)
@@
 			)
 		)
-		(property "Footprint" ""
+		(property "Footprint" "Capacitor_SMD:C_0402_1005Metric"
 			(at 100.33 144.78 0)
 			(hide yes)
@@
 			)
 		)
-		(property "Footprint" ""
+		(property "Footprint" "Capacitor_SMD:C_0402_1005Metric"
 			(at 281.94 30.48 0)
 			(hide yes)
@@
 			)
 		)
-		(property "Footprint" ""
+		(property "Footprint" "Capacitor_SMD:C_0402_1005Metric"
 			(at 92.71 30.48 0)
 			(hide yes)
@@
 			)
 		)
-		(property "Footprint" ""
+		(property "Footprint" "Capacitor_SMD:C_0402_1005Metric"
 			(at 120.65 144.78 0)
 			(hide yes)
@@
 			)
 		)
-		(property "Footprint" ""
+		(property "Footprint" "Capacitor_SMD:C_0402_1005Metric"
 			(at 160.02 30.48 0)
 			(hide yes)
@@
 			)
 		)
-		(property "Footprint" ""
+		(property "Footprint" "Resistor_SMD:R_0402_1005Metric"
 			(at 109.22 198.12 0)
 			(hide yes)
@@
 			)
 		)
-		(property "Footprint" ""
+		(property "Footprint" "Resistor_SMD:R_0402_1005Metric"
 			(at 36.83 115.57 0)
 			(hide yes)
