File: lmx2594.kicad_sch (KiCad schematic)
At the start: 50 parts, among them J28 SYSREFREQ, J29 TUNESENSE, U20 LMX2594

Commit message: add NC and fix ERC
Connections:
- net +3.3VA_LMXDIG is gone; now on net VCC_DIG: R121.2, R123.2
Other:
- sheet Linear POL LMX ports: added none; removed ILIM-
- sheet Linear POL LMX BUF ports: added none; removed ILIM-
