File: huskypointofload.kicad_sch (KiCad schematic)
At the start: 20 parts, among them J1 POWER_IN, J10 ADC_C, J11 ADC_D, J12 SYNCOUT, J13 REFOUT, J14 PPSOUT, J2 PMOD, J3 TO_FRIDGE, J4 FROM_FRIDGE, J5 PPSIN, J6 DAC_A, J7 DAC_B, J8 ADC_A, J9 ADC_B

Commit message: Round 2 Review, power tree cleanup
Parts:
- added R1, R2: 4.7k, Resistor_THT:R_Array_SIP4, symbol Device:R_Small
- gave numbers to parts that had none: 1
- renumbered J9 to J10, J10 to J11, J11 to J12, J12 to J13, J13 to J14, J14 to J15, J5 to J6, J6 to J7, J7 to J8, J8 to J9, R1 to R3, R2 to R4, R3 to R5, R4 to R6, R5 to R7
Connections:
- net ~{RF_CS0}: now also R1.2
- net ~{RF_CS1}: now also R2.2
- new net +3.3V: R1.1, R2.1
Other:
- sheet Linear POL LMK VCO renamed Linear LO Drive
- sheet Monitor Path ports: added 5V; removed 6V
- sheet RX Mixer ports: added 5V; removed 6V
- sheet TX Mixer ports: added 5V; removed 6V
- note removed: "12VRF"
- note removed: "3.3"
- note removed: "3.3LMKDIG"
- note removed: "3.3LMKVCO"
- note removed: "3.3LMXDIG"
- note removed: "3.3LMXPLL"
- note removed: "3.3LMXVCO"
- note removed: "4V"
- note removed: "5A FUSE + FILTER 250mV/A ISENSE"
- note removed: "LMR36510ADDA 48V/12V->3.3V1A"
- note removed: "LT3045 4V->3.3V0.8A"
- note removed: "LT8625S uMOD 12V->4V8A"
- note removed: "TODO: Update Power Tree TODO: Add Clock Tree"
- note removed: "VBUS"
- note removed: "VDC"

Commit message: Darrel Suggestions
Parts:
- R1, R2: footprint Resistor_THT:R_Array_SIP4 -> (none)
Other:
- note added: "0-2GHz"
- note added: "10us Pulse Driven by FS725"
- note added: "256MHz"
- note added: "3-8.5GHz"
- note added: "3.5-18GHz (flatness over 4-8 Prioritized)"
- note added: "3.5-8.5GHz"
- note added: "6.5-8.5GHz"
- note added: "8MHz-100MHz"
- moved on the sheet: J1, J2, J3, J4, J5, R1, R2, R3, R4, R5, R6, R7

Commit message: Passive footprint pass
Parts:
- R1, R2, R3, R4, R5: footprint (none) -> Resistor_SMD:R_0402_1005Metric
Changed lines of the file:
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@@
 			)
 		)
-		(property "Footprint" ""
+		(property "Footprint" "Resistor_SMD:R_0402_1005Metric"
 			(at 144.78 205.74 0)
 			(hide yes)
@@
 			)
 		)
-		(property "Footprint" ""
+		(property "Footprint" "Resistor_SMD:R_0402_1005Metric"
 			(at 152.4 205.74 0)
 			(hide yes)
@@
 			)
 		)
-		(property "Footprint" ""
+		(property "Footprint" "Resistor_SMD:R_0402_1005Metric"
 			(at 50.8 140.97 0)
 			(hide yes)
@@
 			)
 		)
-		(property "Footprint" ""
+		(property "Footprint" "Resistor_SMD:R_0402_1005Metric"
 			(at 53.34 140.97 0)
 			(hide yes)
@@
 			)
 		)
-		(property "Footprint" ""
+		(property "Footprint" "Resistor_SMD:R_0402_1005Metric"
 			(at 154.94 205.74 0)
 			(hide yes)

Commit message: add NC and fix ERC
Parts:
- removed J1: POWER_IN, symbol Connector:Barrel_Jack
- added J1: MINIFIT, Connector_PCBEdge:BUS_PCIexpress_x1, symbol Connector_Generic:Conn_02x02_Counter_Clockwise
Connections:
- net +VDC: now also J1.3 (Pin_3), J1.4 (Pin_4)
- net GND: now also J1.1 (Pin_1), J1.2 (Pin_2)
Other:
- sheet Linear LO Drive ports: added none; removed ILIM-
- sheet MCU ports: added ~{LMX_{LO}CS}; removed none
