File: rx_chain.kicad_sch (KiCad schematic)
At the start: 40 parts, among them U27 ADL8124, U28 ADL6332, U29 ADL6331, U30 MEQ0-20ASM, U31 MC16-0222SM

Commit message: Darrel Suggestions
Parts:
- removed C174, C177, C183: 100n, symbol Device:C_Feedthrough
- added C173: 1n, Capacitor_SMD:C_0201_0603Metric, symbol Device:C_Small
- added C175, C181, C187: 1u, symbol Device:C_Feedthrough
- C178, C179, C180, C184, C185, C186: value 100n -> 1u; DIGIKEY_PN 490-6969-1-ND -> 490-13394-1-ND
- R209, R210, R211, R212, R215, R216, R217, R218: footprint Resistor_THT:R_Array_SIP4 -> (none)
- U30: footprint Package_SO:MSOP-10_3x3mm_P0.5mm -> (none)
- gave numbers to parts that had none: 3
- renumbered C175 to C176, C176 to C177, C181 to C182, C182 to C183
Connections:
- net +3.3VA_LNA: now also C175.3
- net GND: now also C175.2, C181.2, C187.2
- net Linear POL LMK VCO/KELVIN: now also C175.1
- net RFIN: now also C173.2; no longer U27.4 (VTEMP)
- net VCC_AMP1: now also C181.1
- net VCC_AMP2: now also C187.1
- net at R218.1: now also C187.3; no longer C186.3
- net at C184.3: now also R215.1; no longer R216.1
- net at R217.1: now also C186.3; no longer C185.3
- net at R210.1: now also C179.3; no longer C178.3
- net at R211.1: now also C180.3; no longer C179.3
- net at R212.1: now also C181.3; no longer C180.3
- net at R209.1: now also C178.3
- new net: C173.1, U27.4 (VTEMP)
- new net: C185.3, R216.1

Commit message: Passive footprint pass
Parts:
- C172, C174: footprint (none) -> Capacitor_SMD:C_0402_1005Metric
- R206, R209, R210, R211, R212, R215, R216, R217, R218: footprint (none) -> Resistor_SMD:R_0402_1005Metric
Changed lines of the file:
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@@
 			)
 		)
-		(property "Footprint" ""
+		(property "Footprint" "Capacitor_SMD:C_0402_1005Metric"
 			(at 60.96 71.12 0)
 			(hide yes)
@@
 			)
 		)
-		(property "Footprint" ""
+		(property "Footprint" "Resistor_SMD:R_0402_1005Metric"
 			(at 320.04 96.52 0)
 			(hide yes)
@@
 			)
 		)
-		(property "Footprint" ""
+		(property "Footprint" "Resistor_SMD:R_0402_1005Metric"
 			(at 180.34 50.8 0)
 			(hide yes)
@@
 			)
 		)
-		(property "Footprint" ""
+		(property "Footprint" "Resistor_SMD:R_0402_1005Metric"
 			(at 320.04 73.66 0)
 			(hide yes)
@@
 			)
 		)
-		(property "Footprint" ""
+		(property "Footprint" "Resistor_SMD:R_0402_1005Metric"
 			(at 82.55 187.96 0)
 			(hide yes)
@@
 			)
 		)
-		(property "Footprint" ""
+		(property "Footprint" "Resistor_SMD:R_0402_1005Metric"
 			(at 180.34 96.52 0)
 			(hide yes)
@@
 			)
 		)
-		(property "Footprint" ""
+		(property "Footprint" "Resistor_SMD:R_0402_1005Metric"
 			(at 180.34 73.66 0)
 			(hide yes)
@@
 			)
 		)
-		(property "Footprint" ""
+		(property "Footprint" "Resistor_SMD:R_0402_1005Metric"
 			(at 180.34 27.94 0)
 			(hide yes)
@@
 			)
 		)
-		(property "Footprint" ""
+		(property "Footprint" "Resistor_SMD:R_0402_1005Metric"
 			(at 320.04 50.8 0)
 			(hide yes)
@@
 			)
 		)
-		(property "Footprint" ""
+		(property "Footprint" "Capacitor_SMD:C_0402_1005Metric"
 			(at 35.56 71.12 0)
 			(hide yes)
@@
 			)
 		)
-		(property "Footprint" ""
+		(property "Footprint" "Resistor_SMD:R_0402_1005Metric"
 			(at 320.04 27.94 0)
 			(hide yes)

Commit message: add NC and fix ERC
Parts:
- removed TP10: TPRXOUT, Connector_Coaxial:CoaxialSwitch_Hirose_MS-156C3_Horizontal, symbol Connector:CoaxialSwitch_Testpoint
- added C305: 1n, Capacitor_SMD:C_0201_0603Metric, symbol Device:C_Small
- added R275: 100, Resistor_SMD:R_0402_1005Metric, symbol Device:R_Small
- added TP10: TPG, Relay_THT:Relay_DPDT_Schrack-RT2-FormC_RM5mm, symbol Connector:TestPoint_Small
Connections:
- net RF Switching PSU/PGFB+ is gone; now on net +4V_RX: R204.1
- net CIPO: now also R275.2; no longer U28.18 (SDO)
- net GND: now also U28.13 (ATT0), U28.6 (ATT1), U29.13 (ATT0), U29.6 (ATT1), TP10.1; no longer U27.8 (GND)
- net VCC_AMP1: now also R209.1, R210.1, R211.1, R212.1; no longer C178.1, C179.1, C180.1, C181.1
- net VCC_AMP1_AMP1: now also C178.3; no longer R209.2
- net VCC_AMP1_AMP1A: now also C179.3; no longer R210.2
- net VCC_AMP1_AMP2: now also C180.3; no longer R211.2
- net VCC_AMP1_AMP2A: now also C181.3; no longer R212.2
- net VCC_AMP2: now also R215.1, R216.1, R217.1, R218.1; no longer C184.1, C185.1, C186.1, C187.1
- net VCC_AMP2_AMP1: now also C184.3; no longer R215.2
- net VCC_AMP2_AMP1A: now also C185.3; no longer R216.2
- net VCC_AMP2_AMP2: now also C186.3; no longer R217.2
- net VCC_AMP2_AMP2A: now also C187.3; no longer R218.2
- net VCC_RX_DIG: now also U28.22 (VCC_{FUSE}), U29.22 (VCC_{FUSE}); no longer U28.11 (VCC_{FUSE}), U29.11 (VCC_{FUSE})
- net VTEMP_AMP0: now also U27.2 (VTEMP); no longer U27.4 (VTEMP)
- net at U31.5 (RFIN): now also C305.1
- net at U30.9 (RFOUT): now also C305.2
- new net: C187.1, R218.2
- new net: C180.1, R211.2
- new net: C179.1, R210.2
- new net: R275.1, U28.18 (SDO)
- new net: C184.1, R215.2
- new net: C186.1, R217.2
- new net: C181.1, R212.2
- new net: C178.1, R209.2
- new net: C185.1, R216.2
- no-connect marks 8 -> 4
Other:
- sheet Linear POL AMP1 ports: added none; removed ILIM-
- sheet Linear POL LMK AMP2 ports: added none; removed ILIM-
- sheet Linear POL LMK VCO ports: added none; removed ILIM-
- sheet RF Switching PSU ports: added none; removed PGFB+
- note added: "For Solderin Coax Probe"
- moved on the sheet: C178, C179, C180, C181, C184, C185, C186, C187, R209, R210, R211, R212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
